File: hardware/ESP32-P4_16.kicad_pcb (KiCad board)
At the start: 2 copper layers, 151.1 x 93.4 mm, 99 parts, among them J1 String1, J10 String10, J11 String11, J12 String12, J13 String13, J14 String14, J15 String15, J16 String16, J17 Power In Left, J18 Power In Right, J19 GPIO, J2 String2, J22 DMX1, J26 OLED, J27 Aux Pwr, J28 VIN Select, J3 String3, J4 String4, J5 String5, J6 String6, J7 String7, J8 String8, J9 String9, SW1 Enter BTN, SW2 Down BTN, U1 ESP32-P4-ETH, U2 L7805, U4 74HCT541, U5 UA9638CP, U6 74HCT541, U7 LMR38020SDDAR

Commit message: Add CI firmware build; HW1/HW2 pin options; SD/PSRAM/OTA fixes
CI: .github/workflows/build-firmware.yml builds both HW variants with
arduino-cli (esp32:esp32:esp32p4:PSRAM=enabled) and uploads the .bin
artifacts. NOTE: firmware must be built with PSRAM=enabled — the board's
PSRAM defaults to Disabled, which left getPsramSize()=0.

Firmware:
- HW_VERSION build switch: HW1 (default) = original pins; HW2 (-DHW_VERSION=2)
  reroutes pixel ports 12-16 to GPIO32,33,46,47,48 (off the USB pins), per the
  revised schematic.
- SD: use the esp32p4 variant's auto-config (SLOT-0 IOMUX, LDO ch4, power pin)
  instead of custom setPins/power handling; only mount in FSEQ mode so it can't
  disturb PARLIO in E1.31/DDP. (Card still not mounting — needs serial-log
  diagnosis; sdError exposed in /api/status.)
- OTA: reliable streaming path (throttle the client to avoid the AsyncTCP
  heap-exhaustion reset); PSRAM-buffered variant removed (crashes under heavy
  Ethernet RX).
- /api/status diagnostics: parlioOk, menuActive, b1HeldMs, otaMode, freePsram,
  psramSize, sdError.

Hardware: HW2 schematic (ports 12-16 remap, USB pins now NC).

Co-Authored-By: Claude Opus 4.8 (1M context) <noreply@anthropic.com>
Connections:
- U1 pad 19: DATA14 -> unconnected-(U1-DM/GPIO24-Pad19)
- U1 pad 20: DATA16 -> unconnected-(U1-DP/GPIO25-Pad20)
- U1 pad 21: DATA15 -> DATA16
- U1 pad 22: DATA13 -> DATA15
- U1 pad 24: DATA12 -> DATA14
- U1 pad 25: unconnected-(U1-GPIO33-Pad25) -> DATA13
- U1 pad 26: unconnected-(U1-GPIO32-Pad26) -> DATA12
Routing:
- net DATA16: track 12.2 -> 31.1 mm
- net DATA14: track 11.0 -> 29.8 mm
- net BTN1: track 62.0 -> 72.4 mm, vias 0 -> 2
- net DATA12: track 28.2 -> 30.4 mm
- net I2C_SDA: track 79.9 -> 81.1 mm, vias 0 -> 1
- net DATA13: track 29.0 -> 29.6 mm
