File: hardware/ESP32-P4_16.kicad_pcb (KiCad board)
At the start: 2 copper layers, 151.1 x 93.4 mm, 99 parts, among them J1 String1, J10 String10, J11 String11, J12 String12, J13 String13, J14 String14, J15 String15, J16 String16, J17 Power In Left, J18 Power In Right, J19 GPIO, J2 String2, J22 DMX1, J26 OLED, J27 Aux Pwr, J28 VIN Select, J3 String3, J4 String4, J5 String5, J6 String6, J7 String7, J8 String8, J9 String9, SW1 Enter BTN, SW2 Down BTN, U1 ESP32-P4-ETH, U2 L7805, U4 74HCT541, U5 UA9638CP, U6 74HCT541, U7 LMR38020SDDAR

Commit message: Update PCB layout
Co-Authored-By: Claude Opus 4.8 (1M context) <noreply@anthropic.com>
Parts:
- moved R2 2.33 mm to (86.6, 103.2)
- moved U5 0.70 mm to (92.5, 103.1)
- moved R9 0.61 mm to (84.0, 110.6)
- moved R10 0.61 mm to (84.0, 107.2)
- moved C9 0.60 mm to (97.2, 105.7)
Routing:
- net /Serial/DMX1+: track 16.5 -> 15.0 mm
- net GND: track 48.3 -> 49.3 mm
- net Net-(R10-Pad1): track 50.8 -> 51.4 mm
- net V_DMX: track 21.3 -> 22.0 mm

Commit message: Update PCB layout
Co-Authored-By: Claude Opus 4.8 (1M context) <noreply@anthropic.com>
Parts:
- moved J19 5.15 mm to (75.6, 75.1)
- moved R8 4.96 mm to (83.0, 73.0)
Routing:
- net GND: track 49.3 -> 56.2 mm
- net Net-(R10-Pad1): track 51.4 -> 57.9 mm
- net VIN1_ADC: track 63.6 -> 60.9 mm
- net GPIO23: track 75.6 -> 74.7 mm
- net GPIO22: track 74.3 -> 73.8 mm
