File: hardware/ESP32.kicad_sch (KiCad schematic)
At the start: 1 part, among them U1 ESP32-P4-ETH

Commit message: Add CI firmware build; HW1/HW2 pin options; SD/PSRAM/OTA fixes
CI: .github/workflows/build-firmware.yml builds both HW variants with
arduino-cli (esp32:esp32:esp32p4:PSRAM=enabled) and uploads the .bin
artifacts. NOTE: firmware must be built with PSRAM=enabled — the board's
PSRAM defaults to Disabled, which left getPsramSize()=0.

Firmware:
- HW_VERSION build switch: HW1 (default) = original pins; HW2 (-DHW_VERSION=2)
  reroutes pixel ports 12-16 to GPIO32,33,46,47,48 (off the USB pins), per the
  revised schematic.
- SD: use the esp32p4 variant's auto-config (SLOT-0 IOMUX, LDO ch4, power pin)
  instead of custom setPins/power handling; only mount in FSEQ mode so it can't
  disturb PARLIO in E1.31/DDP. (Card still not mounting — needs serial-log
  diagnosis; sdError exposed in /api/status.)
- OTA: reliable streaming path (throttle the client to avoid the AsyncTCP
  heap-exhaustion reset); PSRAM-buffered variant removed (crashes under heavy
  Ethernet RX).
- /api/status diagnostics: parlioOk, menuActive, b1HeldMs, otaMode, freePsram,
  psramSize, sdError.

Hardware: HW2 schematic (ports 12-16 remap, USB pins now NC).

Co-Authored-By: Claude Opus 4.8 (1M context) <noreply@anthropic.com>
Connections:
- net DATA12: now also U1.26 (GPIO32); no longer U1.24 (GPIO46)
- net DATA13: now also U1.25 (GPIO33); no longer U1.22 (GPIO47)
- net DATA14: now also U1.24 (GPIO46); no longer U1.19 (DM/GPIO24)
- net DATA15: now also U1.22 (GPIO47); no longer U1.21 (GPIO48)
- net DATA16: now also U1.21 (GPIO48); no longer U1.20 (DP/GPIO25)
