File: hardware/ESP32-P4_16.kicad_sch (KiCad schematic)
At the start: 41 parts, among them J17 Power In Left, J18 Power In Right, J19 GPIO, J26 OLED, J27 Aux Pwr, J28 VIN Select, SW1 Enter BTN, SW2 Down BTN, U2 L7805, U7 LMR38020SDDAR

Commit message: update to new connectors
Parts:
- SW1: value Enter BTN -> Test
- SW2: value Down BTN -> Setup
Changed lines of the file:
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@@
 			)
 		)
-		(property "Value" "Enter BTN"
+		(property "Value" "Test"
 			(at 200.6092 144.653 90)
 			(show_name no)
@@
 			)
 		)
-		(property "Value" "Down BTN"
+		(property "Value" "Setup"
 			(at 217.1192 144.399 90)
 			(show_name no)
