File: hardware/Output1_8.kicad_sch (KiCad schematic)
At the start: 26 parts, among them J1 String1, J2 String2, J3 String3, J4 String4, J5 String5, J6 String6, J7 String7, J8 String8, U6 74HCT541

Commit message: update to new connectors
Parts:
- J1, J2, J3, J4, J5, J6, J7, J8: footprint Scotts:DG250-3.5-03P -> 1864299:PHOENIX_1864299_1
Changed lines of the file:
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@@
 			)
 		)
-		(property "Footprint" "Scotts:DG250-3.5-03P"
+		(property "Footprint" "1864299:PHOENIX_1864299_1"
 			(at 151.13 101.6 0)
 			(hide yes)
@@
 			)
 		)
-		(property "Footprint" "Scotts:DG250-3.5-03P"
+		(property "Footprint" "1864299:PHOENIX_1864299_1"
 			(at 162.56 101.6 0)
 			(hide yes)
@@
 			)
 		)
-		(property "Footprint" "Scotts:DG250-3.5-03P"
+		(property "Footprint" "1864299:PHOENIX_1864299_1"
 			(at 173.99 101.6 0)
 			(hide yes)
@@
 			)
 		)
-		(property "Footprint" "Scotts:DG250-3.5-03P"
+		(property "Footprint" "1864299:PHOENIX_1864299_1"
 			(at 185.42 101.6 0)
 			(hide yes)
@@
 			)
 		)
-		(property "Footprint" "Scotts:DG250-3.5-03P"
+		(property "Footprint" "1864299:PHOENIX_1864299_1"
 			(at 196.85 101.6 0)
 			(hide yes)
@@
 			)
 		)
-		(property "Footprint" "Scotts:DG250-3.5-03P"
+		(property "Footprint" "1864299:PHOENIX_1864299_1"
 			(at 208.28 101.6 0)
 			(hide yes)
@@
 			)
 		)
-		(property "Footprint" "Scotts:DG250-3.5-03P"
+		(property "Footprint" "1864299:PHOENIX_1864299_1"
 			(at 219.71 101.6 0)
 			(hide yes)
@@
 			)
 		)
-		(property "Footprint" "Scotts:DG250-3.5-03P"
+		(property "Footprint" "1864299:PHOENIX_1864299_1"
 			(at 231.14 101.6 0)
 			(hide yes)
