File: hardware/Output9_16.kicad_sch (KiCad schematic)
At the start: 26 parts, among them J10 String10, J11 String11, J12 String12, J13 String13, J14 String14, J15 String15, J16 String16, J9 String9, U4 74HCT541

Commit message: update to new connectors
Parts:
- J10, J11, J12, J13, J14, J15, J16, J9: footprint Scotts:DG250-3.5-03P -> 1864299:PHOENIX_1864299_1
Changed lines of the file:
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@@
 			)
 		)
-		(property "Footprint" "Scotts:DG250-3.5-03P"
+		(property "Footprint" "1864299:PHOENIX_1864299_1"
 			(at 163.83 97.79 0)
 			(hide yes)
@@
 			)
 		)
-		(property "Footprint" "Scotts:DG250-3.5-03P"
+		(property "Footprint" "1864299:PHOENIX_1864299_1"
 			(at 175.26 97.79 0)
 			(hide yes)
@@
 			)
 		)
-		(property "Footprint" "Scotts:DG250-3.5-03P"
+		(property "Footprint" "1864299:PHOENIX_1864299_1"
 			(at 186.69 97.79 0)
 			(hide yes)
@@
 			)
 		)
-		(property "Footprint" "Scotts:DG250-3.5-03P"
+		(property "Footprint" "1864299:PHOENIX_1864299_1"
 			(at 198.12 97.79 0)
 			(hide yes)
@@
 			)
 		)
-		(property "Footprint" "Scotts:DG250-3.5-03P"
+		(property "Footprint" "1864299:PHOENIX_1864299_1"
 			(at 209.55 97.79 0)
 			(hide yes)
@@
 			)
 		)
-		(property "Footprint" "Scotts:DG250-3.5-03P"
+		(property "Footprint" "1864299:PHOENIX_1864299_1"
 			(at 220.98 97.79 0)
 			(hide yes)
@@
 			)
 		)
-		(property "Footprint" "Scotts:DG250-3.5-03P"
+		(property "Footprint" "1864299:PHOENIX_1864299_1"
 			(at 232.41 97.79 0)
 			(hide yes)
@@
 			)
 		)
-		(property "Footprint" "Scotts:DG250-3.5-03P"
+		(property "Footprint" "1864299:PHOENIX_1864299_1"
 			(at 243.84 97.79 0)
 			(hide yes)
